Commit message: xmacrosss  e include

File: dev_ws/src/robot_description/urdf/body.urdf.xacro (robot description, xacro)
@@ -1,23 +1,23 @@
 <?xml version="1.0"?>
 <robot xmlns:xacro="http://www.ros.org/wiki/xacro" name="robot">
-    <material name="body_front_color">
+    <material name="color_body_front">
         <color rgba="1 0.3 0.1 1"/>
     </material>
-    <link name="world"></link>
-    <link name="base">
+    <link name="link_world"></link>
+    <link name="link_base">
         <visual>
-            <origin xyz="2 0 0" rpy="1.57 0 0"/>
+            <origin xyz="0 0 -0.142" rpy="1.57 0 0"/>
             <geometry>
                 <box size="5 0.1 3" />
             </geometry>
-            <material name="body_front_color" />
+            <material name="color_body_front" />
         </visual>
     </link>
-    <joint name="world_to_base" type="fixed">
-        <parent link="world"/>
-        <child link="base"/>
+    <joint name="link_world_to_link_base_joint" type="fixed">
+        <parent link="link_world"/>
+        <child link="link_base"/>
         <origin xyz="0 0 0" rpy="0 0 0"/>
     </joint>
-    <link name="body_front">
+    <link name="link_body_front">
         <visual>
             <origin xyz="0.0 0.0 0.0" rpy="0.0 0.0 0.0"/>
@@ -26,11 +26,47 @@
                     <mesh filename="package://robot_description/meshes/body_front.stl" scale="1.0 1.0 1.0"/>
                 </geometry>
-            <material name="body_front_color" />
+            <material name="color_body_front" />
         </visual>
     </link>
-    <joint name="base_to_body_front" type="fixed">
-        <parent link="base"/>
-        <child link="body_front"/>
-        <origin xyz="0 0 0.1" rpy="0 0 0"/>
+    <link name="link_body_rear">
+        <visual>
+            <origin xyz="0.0 0.0 0.0" rpy="0.0 0.0 0.0"/>
+                <geometry>
+                    <!-- <cylinder radius="0.5" length="1.0"/> -->
+                    <mesh filename="package://robot_description/meshes/body_rear.stl" scale="1.0 1.0 1.0"/>
+                </geometry>
+            <material name="color_body_front" />
+        </visual>
+    </link>
+    <joint name="joint_link_body_front_to_link_body_rear" type="fixed">
+        <parent link="link_body_front"/>
+        <child link="link_body_rear"/>
+        <origin xyz="0.0 0.0 0.0" rpy="0.0 0.0 0.0"/>
     </joint>
+    <link name="link_window">
+        <visual>
+            <origin xyz="0.0 0.0 0.0" rpy="0.0 0.0 0.0"/>
+            <geometry>
+                <mesh filename="package://robot_description/meshes/body_front_window.stl" scale="1.0 1.0 1.0"/>
+            </geometry>
+            <material name="color_body_front" />
+        </visual>
+    </link>
+    <joint name="joint_link_body_front_to_link_window" type="fixed">
+        <parent link="link_body_front"/>
+        <child link="link_window"/>
+        <origin xyz="0.0 0.0 0.0" rpy="0.0 0.0 0.0"/>
+    </joint>
+    <xacro:include filename="wheel.urdf.xacro"/>
+    <xacro:wheel roll="1.57" pitch="0.0" yaw="0.0" x="0.162" y="0.132" z="-0.041"/>
+    <!-- <joint name="link_body_front_to_link_base" type="fixed">
+        <parent link="link_body_front"/>
+        <child link="link_world_to_link_base"/>
+        <origin xyz="0.0 0.0 0.0" rpy="0.0 0.0 0.0"/>
+    </joint> -->
+    <!-- <xacro:wheel_with_joint wheel_name="front_left" roll="1.57" pitch="0.0" yaw="0.0" x="0.162" y="0.132" z="-0.041"/>
+    <xacro:wheel_with_joint wheel_name="front_right" roll="1.57" pitch="0.0" yaw="0.0" x="0.162" y="-0.132" z="-0.041"/>
+    <xacro:wheel_with_joint wheel_name="rear_left" roll="1.57" pitch="0.0" yaw="0.0" x="-0.162" y="0.132" z="-0.041"/>
+    <xacro:wheel_with_joint wheel_name="rear_right" roll="1.57" pitch="0.0" yaw="0.0" x="-0.162" y="-0.132" z="-0.041"/>
+ -->
 </robot>

Commit message: fix display launch

File: dev_ws/src/robot_description/urdf/body.urdf.xacro (robot description, xacro)
@@ -1,9 +1,10 @@
 <?xml version="1.0"?>
 <robot xmlns:xacro="http://www.ros.org/wiki/xacro" name="robot">
+    <xacro:include filename="wheel.urdf.xacro"/>
     <material name="color_body_front">
         <color rgba="1 0.3 0.1 1"/>
     </material>
     <link name="link_world"></link>
-    <link name="link_base">
+    <!-- <link name="link_base">
         <visual>
             <origin xyz="0 0 -0.142" rpy="1.57 0 0"/>
@@ -17,4 +18,9 @@
         <parent link="link_world"/>
         <child link="link_base"/>
+        <origin xyz="0 0 0" rpy="0 0 0"/>
+    </joint> -->
+    <joint name="link_world_to_link_body_front" type="fixed">
+        <parent link="link_world"/>
+        <child link="link_body_front"/>
         <origin xyz="0 0 0" rpy="0 0 0"/>
     </joint>
@@ -58,11 +64,26 @@
         <origin xyz="0.0 0.0 0.0" rpy="0.0 0.0 0.0"/>
     </joint>
-    <xacro:include filename="wheel.urdf.xacro"/>
-    <xacro:wheel roll="1.57" pitch="0.0" yaw="0.0" x="0.162" y="0.132" z="-0.041"/>
-    <!-- <joint name="link_body_front_to_link_base" type="fixed">
+    <xacro:wheel diff_name="front_left" roll="1.57" pitch="0.0" yaw="0.0" x="0.162" y="0.132" z="-0.041"/>
+    <!-- <xacro:wheel diff_name="front_right" roll="-1.57" pitch="0.0" yaw="0.0" x="0.162" y="-0.132" z="-0.041"/>
+    <xacro:wheel diff_name="back_left" roll="1.57" pitch="0.0" yaw="0.0" x="-0.18" y="0.132" z="-0.041"/>
+    <xacro:wheel diff_name="back_right" roll="-1.57" pitch="0.0" yaw="0.0" x="-0.18" y="-0.132" z="-0.041"/>
+     -->
+    <joint name="joint_whell_body_to_front_left" type="continuous">
         <parent link="link_body_front"/>
-        <child link="link_world_to_link_base"/>
+        <child link="link_tire_front_left"/>
+        <axis xyz="0 0 0"/>
+        <origin xyz="0 0 0" rpy="0 0 0"/>
+    </joint>
+    <joint name="joint_rims_to_body" type="fixed">
+        <parent link="link_body_front"/>
+        <child link="link_rims_front_left"/>
+        <origin xyz="0 0 0" rpy="0 0 0"/>
+    </joint>
+    <!-- <joint name="joint_link_body_front_to_link_base" type="fixed">
+        <parent link="link_body_front"/>
+        <child link="link_base"/>
         <origin xyz="0.0 0.0 0.0" rpy="0.0 0.0 0.0"/>
-    </joint> -->
+    </joint>
+     -->
     <!-- <xacro:wheel_with_joint wheel_name="front_left" roll="1.57" pitch="0.0" yaw="0.0" x="0.162" y="0.132" z="-0.041"/>
     <xacro:wheel_with_joint wheel_name="front_right" roll="1.57" pitch="0.0" yaw="0.0" x="0.162" y="-0.132" z="-0.041"/>

File: dev_ws/src/robot_description/urdf/wheel.urdf.xacro (robot description, xacro)
@@ -1,6 +1,6 @@
 <?xml version="1.0"?>
 <robot xmlns:xacro="http://www.ros.org/wiki/xacro">
-    <xacro:macro name="wheel" params="roll pitch yaw x y z">
-        <link name="link_tire">
+    <xacro:macro name="wheel" params="diff_name roll pitch yaw x y z">
+        <link name="link_tire_${diff_name}">
             <visual>
                 <origin xyz="${x} ${y} ${z}" rpy="${roll} ${pitch} ${yaw}"/>
@@ -11,5 +11,5 @@
             </visual>
         </link>
-        <link name="link_rims">
+        <link name="link_rims_${diff_name}">
             <visual>
                 <origin xyz="${x} ${y} ${z}" rpy="${roll} ${pitch} ${yaw}"/>
@@ -20,12 +20,12 @@
             </visual>
         </link>
+        <joint name="joint_link_rims_to_link_tire" type="fixed">
+            <parent link="link_rims_${diff_name}"/>
+            <child link="link_tire_${diff_name}"/>
+            <origin xyz="0.0 0.0 0.0" rpy="0.0 0.0 0.0"/>
+        </joint>
     </xacro:macro>
+    <!-- <xacro:wheel diff_name="left" roll="0.0" pitch="1.57" yaw="0.0" x="0.0" y="0.0" z="0.0"/> -->
     <!-- <xacro:wheel roll="0.0" pitch="1.57" yaw="0.0" x="0.0" y="0.0" z="0.0"/> -->
-    <joint name="joint_link_rims_to_link_tire" type="fixed">
-        <parent link="link_rims"/>
-        <child link="link_tire"/>
-        <origin xyz="0.0 0.0 0.0" rpy="0.0 0.0 0.0"/>
-    </joint>
-    <xacro:wheel roll="0.0" pitch="1.57" yaw="0.0" x="0.0" y="0.0" z="0.0"/>
     <!-- <xacro:macro name="wheel_with_joint" params="wheel_name roll pitch yaw x y z">
         <xacro:wheel roll="${roll}" pitch="${pitch}" yaw="${yaw}" x="${x}" y="${y}" z="${z}"/>

Commit message: rodas não estão A RODAR VER SE É A JOINT COM O MUNDOgit add .git add .git add .git add .git add .git add .git add .git add .git add .git add .git add .git add .

File: dev_ws/src/robot_description/urdf/body.urdf.xacro (robot description, xacro)
@@ -1,93 +1,30 @@
 <?xml version="1.0"?>
-<robot xmlns:xacro="http://www.ros.org/wiki/xacro" name="robot">
-    <xacro:include filename="wheel.urdf.xacro"/>
-    <material name="color_body_front">
-        <color rgba="1 0.3 0.1 1"/>
-    </material>
-    <link name="link_world"></link>
-    <!-- <link name="link_base">
-        <visual>
-            <origin xyz="0 0 -0.142" rpy="1.57 0 0"/>
-            <geometry>
-                <box size="5 0.1 3" />
-            </geometry>
-            <material name="color_body_front" />
-        </visual>
-    </link>
-    <joint name="link_world_to_link_base_joint" type="fixed">
-        <parent link="link_world"/>
-        <child link="link_base"/>
-        <origin xyz="0 0 0" rpy="0 0 0"/>
-    </joint> -->
-    <joint name="link_world_to_link_body_front" type="fixed">
-        <parent link="link_world"/>
-        <child link="link_body_front"/>
-        <origin xyz="0 0 0" rpy="0 0 0"/>
-    </joint>
-    <link name="link_body_front">
+<robot xmlns:xacro="http://www.ros.org/wiki/xacro">
+    <!-- Main body -->
+    <link name="link_body">
+        <!-- Body Front  -->
         <visual>
             <origin xyz="0.0 0.0 0.0" rpy="0.0 0.0 0.0"/>
                 <geometry>
-                    <!-- <cylinder radius="0.5" length="1.0"/> -->
                     <mesh filename="package://robot_description/meshes/body_front.stl" scale="1.0 1.0 1.0"/>
                 </geometry>
             <material name="color_body_front" />
         </visual>
-    </link>
-    <link name="link_body_rear">
+        <!-- Body Rear -->
         <visual>
             <origin xyz="0.0 0.0 0.0" rpy="0.0 0.0 0.0"/>
                 <geometry>
-                    <!-- <cylinder radius="0.5" length="1.0"/> -->
                     <mesh filename="package://robot_description/meshes/body_rear.stl" scale="1.0 1.0 1.0"/>
                 </geometry>
             <material name="color_body_front" />
         </visual>
-    </link>
-    <joint name="joint_link_body_front_to_link_body_rear" type="fixed">
-        <parent link="link_body_front"/>
-        <child link="link_body_rear"/>
-        <origin xyz="0.0 0.0 0.0" rpy="0.0 0.0 0.0"/>
-    </joint>
-    <link name="link_window">
+        <!-- Body Window -->
         <visual>
             <origin xyz="0.0 0.0 0.0" rpy="0.0 0.0 0.0"/>
-            <geometry>
-                <mesh filename="package://robot_description/meshes/body_front_window.stl" scale="1.0 1.0 1.0"/>
-            </geometry>
+                <geometry>
+                    <mesh filename="package://robot_description/meshes/body_front_window.stl" scale="1.0 1.0 1.0"/>
+                </geometry>
             <material name="color_body_front" />
         </visual>
     </link>
-    <joint name="joint_link_body_front_to_link_window" type="fixed">
-        <parent link="link_body_front"/>
-        <child link="link_window"/>
-        <origin xyz="0.0 0.0 0.0" rpy="0.0 0.0 0.0"/>
-    </joint>
-    <xacro:wheel diff_name="front_left" roll="1.57" pitch="0.0" yaw="0.0" x="0.162" y="0.132" z="-0.041"/>
-    <!-- <xacro:wheel diff_name="front_right" roll="-1.57" pitch="0.0" yaw="0.0" x="0.162" y="-0.132" z="-0.041"/>
-    <xacro:wheel diff_name="back_left" roll="1.57" pitch="0.0" yaw="0.0" x="-0.18" y="0.132" z="-0.041"/>
-    <xacro:wheel diff_name="back_right" roll="-1.57" pitch="0.0" yaw="0.0" x="-0.18" y="-0.132" z="-0.041"/>
-     -->
-    <joint name="joint_whell_body_to_front_left" type="continuous">
-        <parent link="link_body_front"/>
-        <child link="link_tire_front_left"/>
-        <axis xyz="0 0 0"/>
-        <origin xyz="0 0 0" rpy="0 0 0"/>
-    </joint>
-    <joint name="joint_rims_to_body" type="fixed">
-        <parent link="link_body_front"/>
-        <child link="link_rims_front_left"/>
-        <origin xyz="0 0 0" rpy="0 0 0"/>
-    </joint>
-    <!-- <joint name="joint_link_body_front_to_link_base" type="fixed">
-        <parent link="link_body_front"/>
-        <child link="link_base"/>
-        <origin xyz="0.0 0.0 0.0" rpy="0.0 0.0 0.0"/>
-    </joint>
-     -->
-    <!-- <xacro:wheel_with_joint wheel_name="front_left" roll="1.57" pitch="0.0" yaw="0.0" x="0.162" y="0.132" z="-0.041"/>
-    <xacro:wheel_with_joint wheel_name="front_right" roll="1.57" pitch="0.0" yaw="0.0" x="0.162" y="-0.132" z="-0.041"/>
-    <xacro:wheel_with_joint wheel_name="rear_left" roll="1.57" pitch="0.0" yaw="0.0" x="-0.162" y="0.132" z="-0.041"/>
-    <xacro:wheel_with_joint wheel_name="rear_right" roll="1.57" pitch="0.0" yaw="0.0" x="-0.162" y="-0.132" z="-0.041"/>
- -->
 </robot>

File: dev_ws/src/robot_description/urdf/wheel.urdf.xacro (robot description, xacro)
@@ -2,5 +2,6 @@
 <robot xmlns:xacro="http://www.ros.org/wiki/xacro">
     <xacro:macro name="wheel" params="diff_name roll pitch yaw x y z">
-        <link name="link_tire_${diff_name}">
+        <link name="link_wheel_${diff_name}">
+            <!-- Mesh para o pneu -->
             <visual>
                 <origin xyz="${x} ${y} ${z}" rpy="${roll} ${pitch} ${yaw}"/>
@@ -10,6 +11,5 @@
                 <material name="color_body_front" />
             </visual>
-        </link>
-        <link name="link_rims_${diff_name}">
+            <!-- Mesh para o RIMS -->
             <visual>
                 <origin xyz="${x} ${y} ${z}" rpy="${roll} ${pitch} ${yaw}"/>
@@ -20,20 +20,4 @@
             </visual>
         </link>
-        <joint name="joint_link_rims_to_link_tire" type="fixed">
-            <parent link="link_rims_${diff_name}"/>
-            <child link="link_tire_${diff_name}"/>
-            <origin xyz="0.0 0.0 0.0" rpy="0.0 0.0 0.0"/>
-        </joint>
     </xacro:macro>
-    <!-- <xacro:wheel diff_name="left" roll="0.0" pitch="1.57" yaw="0.0" x="0.0" y="0.0" z="0.0"/> -->
-    <!-- <xacro:wheel roll="0.0" pitch="1.57" yaw="0.0" x="0.0" y="0.0" z="0.0"/> -->
-    <!-- <xacro:macro name="wheel_with_joint" params="wheel_name roll pitch yaw x y z">
-        <xacro:wheel roll="${roll}" pitch="${pitch}" yaw="${yaw}" x="${x}" y="${y}" z="${z}"/>
-        <joint name="joint_${wheel_name}" type="continuous">
-            <parent link="base_link"/>
-            <child link="link_tire"/>
-            <origin xyz="${x} ${y} ${z}" rpy="${roll} ${pitch} ${yaw}"/>
-        </joint>
-    </xacro:macro> -->
-    <!-- <xacro:wheel_with_joint wheel_name="front_right" roll="1.57" pitch="0.0" yaw="0.0" x="0.162" y="-0.132" z="-0.041"/> -->
 </robot>
