Commit message: GG

File: dev_ws/src/robot_description/urdf/body.urdf.xacro (robot description, xacro)
@@ -3,27 +3,24 @@
     <!-- Main body -->
     <link name="link_body">
-        <!-- Body Front  -->
+        <!-- Body Front -->
         <visual>
-            <origin xyz="0.0 0.0 0.0" rpy="0.0 0.0 0.0"/>
-                <geometry>
-                    <mesh filename="package://robot_description/meshes/body_front.stl" scale="1.0 1.0 1.0"/>
-                </geometry>
-            <material name="color_body_front" />
+            <geometry>
+                <mesh filename="package://robot_description/meshes/body_front.stl" scale="1.0 1.0 1.0"/>
+            </geometry>
+            <material name="color_body_front"/>
         </visual>
         <!-- Body Rear -->
         <visual>
-            <origin xyz="0.0 0.0 0.0" rpy="0.0 0.0 0.0"/>
-                <geometry>
-                    <mesh filename="package://robot_description/meshes/body_rear.stl" scale="1.0 1.0 1.0"/>
-                </geometry>
-            <material name="color_body_front" />
+            <geometry>
+                <mesh filename="package://robot_description/meshes/body_rear.stl" scale="1.0 1.0 1.0"/>
+            </geometry>
+            <material name="color_body_front"/>
         </visual>
         <!-- Body Window -->
         <visual>
-            <origin xyz="0.0 0.0 0.0" rpy="0.0 0.0 0.0"/>
-                <geometry>
-                    <mesh filename="package://robot_description/meshes/body_front_window.stl" scale="1.0 1.0 1.0"/>
-                </geometry>
-            <material name="color_body_front" />
+            <geometry>
+                <mesh filename="package://robot_description/meshes/body_front_window.stl" scale="1.0 1.0 1.0"/>
+            </geometry>
+            <material name="color_body_front"/>
         </visual>
     </link>

File: dev_ws/src/robot_description/urdf/robot.urdf.xacro (robot description, xacro)
@@ -10,57 +10,51 @@
     <xacro:include filename="wheel.urdf.xacro"/>
     <xacro:include filename="body.urdf.xacro"/>
-    <!-- Wheel definitions -->
-    <xacro:property name="wheel_roll" value="1.57"/>
-    <xacro:property name="wheel_pitch" value="0.0"/>
-    <xacro:property name="wheel_yaw" value="0.0"/>
+    <!-- Wheel offsets -->
     <xacro:property name="wheel_offset_y" value="0.132"/>
     <xacro:property name="wheel_offset_z" value="-0.041"/>
     <xacro:property name="wheel_offset_x_f" value="0.162"/>
     <xacro:property name="wheel_offset_x_r" value="-0.18"/>
-    <xacro:wheel diff_name="front_left"
-        roll="${wheel_roll}" pitch="${wheel_pitch}" yaw="${wheel_yaw}"
-        x="0" y="0" z="0"/>
-    <xacro:wheel diff_name="front_right"
-        roll="-${wheel_roll}" pitch="${wheel_pitch}" yaw="${wheel_yaw}"
-        x="0" y="0" z="0"/>
-    <xacro:wheel diff_name="rear_left" roll="${wheel_roll}" pitch="${wheel_pitch}" yaw="${wheel_yaw}"
-        x="0" y="0" z="0"/>
-    <xacro:wheel diff_name="rear_right" roll="-${wheel_roll}" pitch="${wheel_pitch}" yaw="${wheel_yaw}"
-        x="0" y="0" z="0"/>
-    <!-- Joints for wheels -->
-    <xacro:create_wheel_joint wheel_name="front_left" axis_xyz="0 0 1" origin_xyz="${wheel_offset_x_f} ${wheel_offset_y} ${wheel_offset_z}" origin_rpy="0 0 0"/>
-    <xacro:create_wheel_joint wheel_name="front_right" axis_xyz="0 0 1" origin_xyz="${wheel_offset_x_f} -${wheel_offset_y} ${wheel_offset_z}" origin_rpy="0 0 0"/>
-    <xacro:create_wheel_joint wheel_name="rear_left" axis_xyz="0 0 1" origin_xyz="${wheel_offset_x_r} ${wheel_offset_y} ${wheel_offset_z}" origin_rpy="0 0 0"/>
-    <xacro:create_wheel_joint wheel_name="rear_right" axis_xyz="0 0 1" origin_xyz="${wheel_offset_x_r} -${wheel_offset_y} ${wheel_offset_z}" origin_rpy="0 0 0"/>
-    <!-- Joints World -->
+    <xacro:property name="wheel_roll" value="1.57"/>
+    <xacro:property name="wheel_pitch" value="0.0"/>
+    <xacro:property name="wheel_yaw" value="0.0"/>
+    <!-- Define wheels with steering -->
+    <xacro:create_wheel_with_steering
+        wheel_name="front_left"
+        steering_axis_xyz="0 0 1"
+        steering_origin_xyz="${wheel_offset_x_f} ${wheel_offset_y} ${wheel_offset_z}"
+        steering_origin_rpy="0 0 0"
+        wheel_axis_xyz="0 0 1"
+        wheel_origin_xyz="0 0 0"
+        wheel_origin_rpy="${wheel_roll} ${wheel_pitch} ${wheel_yaw}"
+        />
+    <xacro:create_wheel_with_steering
+        wheel_name="front_right"
+        steering_axis_xyz="0 0 1"
+        steering_origin_xyz="${wheel_offset_x_f} -${wheel_offset_y} ${wheel_offset_z}"
+        steering_origin_rpy="0 0 0"
+        wheel_axis_xyz="0 0 1"
+        wheel_origin_xyz="0 0 0"
+        wheel_origin_rpy="-${wheel_roll} ${wheel_pitch} ${wheel_yaw}"/>
+    <xacro:create_wheel_with_steering
+        wheel_name="rear_left"
+        steering_axis_xyz="0 0 1"
+        steering_origin_xyz="${wheel_offset_x_r} ${wheel_offset_y} ${wheel_offset_z}"
+        steering_origin_rpy="0 0 0"
+        wheel_axis_xyz="0 0 1"
+        wheel_origin_xyz="0 0 0"
+        wheel_origin_rpy="${wheel_roll} ${wheel_pitch} ${wheel_yaw}"/>
+    <xacro:create_wheel_with_steering
+        wheel_name="rear_right"
+        steering_axis_xyz="0 0 1"
+        steering_origin_xyz="${wheel_offset_x_r} -${wheel_offset_y} ${wheel_offset_z}"
+        steering_origin_rpy="0 0 0"
+        wheel_axis_xyz="0 0 1"
+        wheel_origin_xyz="0 0 0"
+        wheel_origin_rpy="-${wheel_roll} ${wheel_pitch} ${wheel_yaw}"/>
+    <!-- Fixed joint to world -->
     <joint name="world_to_link_body" type="fixed">
         <parent link="world"/>
         <child link="link_body"/>
-        <axis xyz="0 0 0"/>
         <origin xyz="0 0 0" rpy="0 0 0"/>
     </joint>
-    <!-- <joint name="world_to_wheel_front_left" type="fixed">
-        <parent link="world"/>
-        <child link="link_wheel_front_left"/>
-        <axis xyz="0 0 0"/>
-        <origin xyz="0 0 0" rpy="0 0 0"/>
-    </joint>
-    <joint name="world_to_wheel_front_right" type="fixed">
-        <parent link="world"/>
-        <child link="link_wheel_front_right"/>
-        <axis xyz="0 0 0"/>
-        <origin xyz="0 0 0" rpy="0 0 0"/>
-    </joint>
-    <joint name="world_to_wheel_rear_left" type="fixed">
-        <parent link="world"/>
-        <child link="link_wheel_rear_left"/>
-        <axis xyz="0 0 0"/>
-        <origin xyz="0 0 0" rpy="0 0 0"/>
-    </joint>
-    <joint name="world_to_wheel_rear_right" type="fixed">
-        <parent link="world"/>
-        <child link="link_wheel_rear_right"/>
-        <axis xyz="0 0 0"/>
-        <origin xyz="0 0 0" rpy="0 0 0"/>
-    </joint> -->
 </robot>

File: dev_ws/src/robot_description/urdf/wheel.urdf.xacro (robot description, xacro)
@@ -1,31 +1,40 @@
 <?xml version="1.0"?>
 <robot xmlns:xacro="http://www.ros.org/wiki/xacro">
-    <xacro:macro name="wheel" params="diff_name roll pitch yaw x y z">
-        <link name="link_wheel_${diff_name}">
-            <!-- Mesh para o pneu -->
+    <!-- Macro for creating wheels with steering -->
+    <xacro:macro name="create_wheel_with_steering" params="wheel_name steering_axis_xyz steering_origin_xyz steering_origin_rpy wheel_axis_xyz wheel_origin_xyz wheel_origin_rpy">
+        <!-- Steering Joint -->
+        <joint name="joint_steering_${wheel_name}" type="revolute">
+            <parent link="link_body"/>
+            <child link="link_steering_${wheel_name}"/>
+            <axis xyz="${steering_axis_xyz}"/>
+            <origin xyz="${steering_origin_xyz}" rpy="${steering_origin_rpy}"/>
+            <limit effort="10.0" velocity="1.0" lower="-0.45" upper="0.45"/>
+        </joint>
+        <!-- Steering Link -->
+        <link name="link_steering_${wheel_name}" />
+        <!-- Rotational Joint -->
+        <joint name="joint_rotation_${wheel_name}" type="continuous">
+            <parent link="link_steering_${wheel_name}"/>
+            <child link="link_wheel_${wheel_name}"/>
+            <axis xyz="${wheel_axis_xyz}"/>
+            <origin xyz="${wheel_origin_xyz}" rpy="${wheel_origin_rpy}"/>
+        </joint>
+        <!-- Wheel Link -->
+        <link name="link_wheel_${wheel_name}">
+            <!-- Tire Mesh -->
             <visual>
-                <origin xyz="${x} ${y} ${z}" rpy="${roll} ${pitch} ${yaw}"/>
                 <geometry>
                     <mesh filename="package://robot_description/meshes/tire.stl" scale="1.0 1.0 1.0"/>
                 </geometry>
-                <material name="color_body_front" />
+                <material name="color_body_front"/>
             </visual>
-            <!-- Mesh para o RIMS -->
+            <!-- Rims Mesh -->
             <visual>
-                <origin xyz="${x} ${y} ${z}" rpy="${roll} ${pitch} ${yaw}"/>
                 <geometry>
                     <mesh filename="package://robot_description/meshes/rims.stl" scale="1.0 1.0 1.0"/>
                 </geometry>
-                <material name="color_body_front" />
+                <material name="color_body_front"/>
             </visual>
         </link>
     </xacro:macro>
-    <xacro:macro name="create_wheel_joint" params="wheel_name axis_xyz origin_xyz origin_rpy">
-        <joint name="joint_wheel_body_to_${wheel_name}" type="continuous">
-            <parent link="link_body"/>
-            <child link="link_wheel_${wheel_name}"/>
-            <axis xyz="${axis_xyz}"/>
-            <origin xyz="${origin_xyz}" rpy="${origin_rpy}"/>
-        </joint>
-    </xacro:macro>
 </robot>

Commit message: A

File: dev_ws/src/robot_description/urdf/body.urdf.xacro (robot description, xacro)
@@ -24,4 +24,28 @@
             <material name="color_body_front"/>
         </visual>
+        <!-- Body Front -->
+        <collision>
+            <geometry>
+                <mesh filename="package://robot_description/meshes/body_front.stl" scale="1.0 1.0 1.0"/>
+            </geometry>
+        </collision>
+        <!-- Body Rear -->
+        <collision>
+            <geometry>
+                <mesh filename="package://robot_description/meshes/body_rear.stl" scale="1.0 1.0 1.0"/>
+            </geometry>
+        </collision>
+        <!-- Body Window -->
+        <collision>
+            <geometry>
+                <mesh filename="package://robot_description/meshes/body_front_window.stl" scale="1.0 1.0 1.0"/>
+            </geometry>
+        </collision>
+        <!-- Inertial -->
+        <inertial>
+            <origin xyz="0 0 0" rpy="0 0 0"/>
+            <mass value="10.0"/>
+            <inertia ixx="0.5" ixy="0.0" ixz="0.0" iyy="0.5" iyz="0.0" izz="0.5"/>
+        </inertial>
     </link>
 </robot>

File: dev_ws/src/robot_description/urdf/wheel.urdf.xacro (robot description, xacro)
@@ -36,4 +36,22 @@
                 <material name="color_body_front"/>
             </visual>
+             <!-- Tire Mesh -->
+            <collision>
+                <geometry>
+                    <mesh filename="package://robot_description/meshes/tire.stl" scale="1.0 1.0 1.0"/>
+                </geometry>
+            </collision>
+            <!-- Rims Mesh -->
+            <collision>
+                <geometry>
+                    <mesh filename="package://robot_description/meshes/rims.stl" scale="1.0 1.0 1.0"/>
+                </geometry>
+            </collision>
+            <!-- Inertial -->
+            <inertial>
+                <origin xyz="0 0 0" rpy="0 0 0"/>
+                <mass value="2.0"/>
+                <inertia ixx="0.1" ixy="0.0" ixz="0.0" iyy="0.1" iyz="0.0" izz="0.1"/>
+            </inertial>
         </link>
     </xacro:macro>
