Commit message: rodas FINALMENTE

File: dev_ws/src/robot_description/urdf/robot.urdf.xacro (robot description, xacro)
@@ -11,33 +11,26 @@
     <xacro:include filename="body.urdf.xacro"/>
     <!-- Wheel definitions -->
-    <xacro:wheel diff_name="front_left" roll="1.57" pitch="0.0" yaw="0.0" x="0.162" y="0.132" z="-0.041"/>
-    <xacro:wheel diff_name="front_right" roll="-1.57" pitch="0.0" yaw="0.0" x="0.162" y="-0.132" z="-0.041"/>
-    <xacro:wheel diff_name="rear_left" roll="1.57" pitch="0.0" yaw="0.0" x="-0.18" y="0.132" z="-0.041"/>
-    <xacro:wheel diff_name="rear_right" roll="-1.57" pitch="0.0" yaw="0.0" x="-0.18" y="-0.132" z="-0.041"/>
+    <xacro:property name="wheel_roll" value="1.57"/>
+    <xacro:property name="wheel_pitch" value="0.0"/>
+    <xacro:property name="wheel_yaw" value="0.0"/>
+    <xacro:property name="wheel_offset_y" value="0.132"/>
+    <xacro:property name="wheel_offset_z" value="-0.041"/>
+    <xacro:property name="wheel_offset_x_f" value="0.162"/>
+    <xacro:property name="wheel_offset_x_r" value="-0.18"/>
+    <xacro:wheel diff_name="front_left"
+        roll="${wheel_roll}" pitch="${wheel_pitch}" yaw="${wheel_yaw}"
+        x="0" y="0" z="0"/>
+    <xacro:wheel diff_name="front_right"
+        roll="-${wheel_roll}" pitch="${wheel_pitch}" yaw="${wheel_yaw}"
+        x="0" y="0" z="0"/>
+    <xacro:wheel diff_name="rear_left" roll="${wheel_roll}" pitch="${wheel_pitch}" yaw="${wheel_yaw}"
+        x="0" y="0" z="0"/>
+    <xacro:wheel diff_name="rear_right" roll="-${wheel_roll}" pitch="${wheel_pitch}" yaw="${wheel_yaw}"
+        x="0" y="0" z="0"/>
     <!-- Joints for wheels -->
-    <joint name="joint_wheel_body_to_front_left" type="continuous">
-        <parent link="link_body"/>
-        <child link="link_wheel_front_left"/>
-        <axis xyz="0 0 0"/>
-        <origin xyz="0.162 0.132 -0.041" rpy="1.57 0 0"/>
-    </joint>
-    <joint name="joint_wheel_body_to_front_right" type="continuous">
-        <parent link="link_body"/>
-        <child link="link_wheel_front_right"/>
-        <axis xyz="0 0 0"/>
-        <origin xyz="0 0 0" rpy="0 0 0"/>
-    </joint>
-    <joint name="joint_wheel_body_to_rear_left" type="continuous">
-        <parent link="link_body"/>
-        <child link="link_wheel_rear_left"/>
-        <axis xyz="0 0 0"/>
-        <origin xyz="0 0 0" rpy="0 0 0"/>
-    </joint>
-    <joint name="joint_wheel_body_to_rear_right" type="continuous">
-        <parent link="link_body"/>
-        <child link="link_wheel_rear_right"/>
-        <axis xyz="0 0 0"/>
-        <origin xyz="0 0 0" rpy="0 0 0"/>
-    </joint>
+    <xacro:create_wheel_joint wheel_name="front_left" axis_xyz="0 0 1" origin_xyz="${wheel_offset_x_f} ${wheel_offset_y} ${wheel_offset_z}" origin_rpy="0 0 0"/>
+    <xacro:create_wheel_joint wheel_name="front_right" axis_xyz="0 0 1" origin_xyz="${wheel_offset_x_f} -${wheel_offset_y} ${wheel_offset_z}" origin_rpy="0 0 0"/>
+    <xacro:create_wheel_joint wheel_name="rear_left" axis_xyz="0 0 1" origin_xyz="${wheel_offset_x_r} ${wheel_offset_y} ${wheel_offset_z}" origin_rpy="0 0 0"/>
+    <xacro:create_wheel_joint wheel_name="rear_right" axis_xyz="0 0 1" origin_xyz="${wheel_offset_x_r} -${wheel_offset_y} ${wheel_offset_z}" origin_rpy="0 0 0"/>
     <!-- Joints World -->
     <joint name="world_to_link_body" type="fixed">
@@ -47,5 +40,5 @@
         <origin xyz="0 0 0" rpy="0 0 0"/>
     </joint>
-    <joint name="world_to_wheel_front_left" type="fixed">
+    <!-- <joint name="world_to_wheel_front_left" type="fixed">
         <parent link="world"/>
         <child link="link_wheel_front_left"/>
@@ -70,4 +63,4 @@
         <axis xyz="0 0 0"/>
         <origin xyz="0 0 0" rpy="0 0 0"/>
-    </joint>
+    </joint> -->
 </robot>

File: dev_ws/src/robot_description/urdf/wheel.urdf.xacro (robot description, xacro)
@@ -21,3 +21,11 @@
         </link>
     </xacro:macro>
+    <xacro:macro name="create_wheel_joint" params="wheel_name axis_xyz origin_xyz origin_rpy">
+        <joint name="joint_wheel_body_to_${wheel_name}" type="continuous">
+            <parent link="link_body"/>
+            <child link="link_wheel_${wheel_name}"/>
+            <axis xyz="${axis_xyz}"/>
+            <origin xyz="${origin_xyz}" rpy="${origin_rpy}"/>
+        </joint>
+    </xacro:macro>
 </robot>

Commit message: laa

File: dev_ws/src/robot_description/urdf/robot.urdf.xacro (robot description, xacro)
@@ -1,60 +1,6 @@
 <?xml version="1.0"?>
 <robot xmlns:xacro="http://www.ros.org/wiki/xacro" name="robot">
-    <!-- Material definition -->
-    <material name="color_body_front">
-        <color rgba="1 0.3 0.1 1"/>
-    </material>
-    <!-- Root World -->
-    <link name="world" />
     <!-- Includes -->
-    <xacro:include filename="wheel.urdf.xacro"/>
-    <xacro:include filename="body.urdf.xacro"/>
-    <!-- Wheel offsets -->
-    <xacro:property name="wheel_offset_y" value="0.132"/>
-    <xacro:property name="wheel_offset_z" value="-0.041"/>
-    <xacro:property name="wheel_offset_x_f" value="0.162"/>
-    <xacro:property name="wheel_offset_x_r" value="-0.18"/>
-    <xacro:property name="wheel_roll" value="1.57"/>
-    <xacro:property name="wheel_pitch" value="0.0"/>
-    <xacro:property name="wheel_yaw" value="0.0"/>
-    <!-- Define wheels with steering -->
-    <xacro:create_wheel_with_steering
-        wheel_name="front_left"
-        steering_axis_xyz="0 0 1"
-        steering_origin_xyz="${wheel_offset_x_f} ${wheel_offset_y} ${wheel_offset_z}"
-        steering_origin_rpy="0 0 0"
-        wheel_axis_xyz="0 0 1"
-        wheel_origin_xyz="0 0 0"
-        wheel_origin_rpy="${wheel_roll} ${wheel_pitch} ${wheel_yaw}"
-        />
-    <xacro:create_wheel_with_steering
-        wheel_name="front_right"
-        steering_axis_xyz="0 0 1"
-        steering_origin_xyz="${wheel_offset_x_f} -${wheel_offset_y} ${wheel_offset_z}"
-        steering_origin_rpy="0 0 0"
-        wheel_axis_xyz="0 0 1"
-        wheel_origin_xyz="0 0 0"
-        wheel_origin_rpy="-${wheel_roll} ${wheel_pitch} ${wheel_yaw}"/>
-    <xacro:create_wheel_with_steering
-        wheel_name="rear_left"
-        steering_axis_xyz="0 0 1"
-        steering_origin_xyz="${wheel_offset_x_r} ${wheel_offset_y} ${wheel_offset_z}"
-        steering_origin_rpy="0 0 0"
-        wheel_axis_xyz="0 0 1"
-        wheel_origin_xyz="0 0 0"
-        wheel_origin_rpy="${wheel_roll} ${wheel_pitch} ${wheel_yaw}"/>
-    <xacro:create_wheel_with_steering
-        wheel_name="rear_right"
-        steering_axis_xyz="0 0 1"
-        steering_origin_xyz="${wheel_offset_x_r} -${wheel_offset_y} ${wheel_offset_z}"
-        steering_origin_rpy="0 0 0"
-        wheel_axis_xyz="0 0 1"
-        wheel_origin_xyz="0 0 0"
-        wheel_origin_rpy="-${wheel_roll} ${wheel_pitch} ${wheel_yaw}"/>
-    <!-- Fixed joint to world -->
-    <joint name="world_to_link_body" type="fixed">
-        <parent link="world"/>
-        <child link="link_body"/>
-        <origin xyz="0 0 0" rpy="0 0 0"/>
-    </joint>
+    <xacro:include filename="robot_core.xacro"/>
+    <xacro:include filename="gazebo_control.xacro"/>
 </robot>
