Commit message: Enhance robot simulation setup by adding ROS2 control dependencies, updating launch files, and refining URDF configurations for improved integration with Gazebo.

File: src/robot_description/urdf/gazebo_control.xacro (robot description, xacro)
@@ -1,37 +1,27 @@
 <?xml version="1.0"?>
 <robot xmlns:xacro="http://www.ros.org/wiki/xacro">
-    <!-- <gazebo>
-        <plugin filename="gz-sim-diff-drive-system" name="gz::sim::systems::DiffDrive">
-            <left_joint>joint_steering_front_left</left_joint>
-            <right_joint>joint_steering_right_left</right_joint>
-            <wheel_separation>1.2</wheel_separation>
-            <wheel_radius>0.4</wheel_radius>
-            <odom_publish_frequency>1</odom_publish_frequency>
-            <topic>cmd_vel</topic>
+    <!-- Gazebo Plugin -->
+    <gazebo>
+        <plugin name="gz_ros2_control-system" filename="gz_ros2_control::GazeboSimROS2ControlPlugin">
+            <parameters>$(find robot_description)/config/robot_sim.controller_manager.yaml</parameters>
         </plugin>
     </gazebo>
- -->
     <!-- Gazebo Body Ref -->
     <gazebo reference="link_body">
-        <material>Gazebo/Grey</material>
     </gazebo>
     <!-- Gazebo Wheels Ref -->
     <gazebo reference="link_wheel_front_left">
-        <material>Gazebo/Black</material>
         <mu1 value="0.001"/>
         <mu2 value="0.001"/>
     </gazebo>
     <gazebo reference="link_wheel_front_right">
-        <material>Gazebo/Black</material>
         <mu1 value="0.001"/>
         <mu2 value="0.001"/>
     </gazebo>
     <gazebo reference="link_wheel_rear_left">
-        <material>Gazebo/Black</material>
         <mu1 value="0.001"/>
         <mu2 value="0.001"/>
     </gazebo>
     <gazebo reference="link_wheel_rear_right">
-        <material>Gazebo/Black</material>
         <mu1 value="0.001"/>
         <mu2 value="0.001"/>

File: src/robot_description/urdf/robot.urdf.xacro (robot description, xacro)
@@ -1,6 +1,11 @@
 <?xml version="1.0"?>
 <robot xmlns:xacro="http://www.ros.org/wiki/xacro" name="robot">
-    <!-- Includes -->
+    <!-- Robot Description -->
     <xacro:include filename="robot_core.xacro"/>
-    <!-- <xacro:include filename="gazebo_control.xacro"/> -->
+    <!-- Gazebo Control -->
+    <xacro:if value="$(arg use_gazebo_ros2_control)">
+        <xacro:include filename="gazebo_control.xacro" />
+    </xacro:if>
+    <!-- ROS Control -->
+    <xacro:include filename="ros2_control.xacro"/>
 </robot>

File: src/robot_description/urdf/robot_core.xacro (robot description, xacro)
@@ -14,5 +14,5 @@
         <color rgba="1 1 1 1" />
     </material>
-    <!-- Root link_base -->
+    <!-- Root link_base -->fl_wheel_joint
     <link name="link_base" />
     <!-- Includes -->
