Commit message: Update robot description launch and hooks for improved resource paths and launch arguments

File: src/robot_description/urdf/body.urdf.xacro (robot description, xacro)
@@ -10,4 +10,9 @@
             <material name="color_body_front"/>
         </visual>
+        <!-- <visual>
+            <geometry>
+                <cylinder radius="1" length="5.0"/>
+            </geometry>
+        </visual> -->
         <!-- Body Rear -->
         <visual>

Commit message: Refactor robot description URDF files for improved material definitions and structure; add world plane configuration for simulation.

File: src/robot_description/urdf/body.urdf.xacro (robot description, xacro)
@@ -8,5 +8,5 @@
                 <mesh filename="package://robot_description/meshes/body_front.stl" scale="1.0 1.0 1.0"/>
             </geometry>
-            <material name="color_body_front"/>
+            <material name="Grey"/>
         </visual>
         <!-- <visual>
@@ -20,5 +20,5 @@
                 <mesh filename="package://robot_description/meshes/body_rear.stl" scale="1.0 1.0 1.0"/>
             </geometry>
-            <material name="color_body_front"/>
+            <material name="Grey"/>
         </visual>
         <!-- Body Window -->
@@ -27,5 +27,5 @@
                 <mesh filename="package://robot_description/meshes/body_front_window.stl" scale="1.0 1.0 1.0"/>
             </geometry>
-            <material name="color_body_front"/>
+            <material name="Black"/>
         </visual>
         <!-- Body Front -->
@@ -49,7 +49,7 @@
         <!-- Inertial -->
         <inertial>
-            <origin xyz="0 0 0" rpy="0 0 0"/>
-            <mass value="10.0"/>
-            <inertia ixx="0.5" ixy="0.0" ixz="0.0" iyy="0.5" iyz="0.0" izz="0.5"/>
+            <origin xyz="0 0 0" rpy="0 0 0" />
+            <mass value="1.0" />
+            <inertia ixx="0.126164" ixy="0.0" ixz="0.0" iyy="0.416519" iyz="0.0" izz="0.481014" />
         </inertial>
     </link>

File: src/robot_description/urdf/gazebo_control.xacro (robot description, xacro)
@@ -1,5 +1,5 @@
 <?xml version="1.0"?>
 <robot xmlns:xacro="http://www.ros.org/wiki/xacro">
-    <gazebo>
+    <!-- <gazebo>
         <plugin filename="gz-sim-diff-drive-system" name="gz::sim::systems::DiffDrive">
             <left_joint>joint_steering_front_left</left_joint>
@@ -11,4 +11,5 @@
         </plugin>
     </gazebo>
+ -->
     <!-- Gazebo Body Ref -->
     <gazebo reference="link_body">

File: src/robot_description/urdf/robot_core.xacro (robot description, xacro)
@@ -2,9 +2,18 @@
 <robot xmlns:xacro="http://www.ros.org/wiki/xacro">
     <!-- Material definition -->
-    <material name="color_body_front">
-        <color rgba="1 0.3 0.1 1"/>
+    <material name="Black">
+        <color rgba="0 0 0 1" />
     </material>
-    <!-- Root World -->
-    <link name="world" />
+    <material name="Grey">
+        <color rgba="0.8 0.8 0.8 1" />
+    </material>
+    <material name="Orange">
+        <color rgba="1 0.6 0 1" />
+    </material>
+    <material name="White">
+        <color rgba="1 1 1 1" />
+    </material>
+    <!-- Root link_base -->
+    <link name="link_base" />
     <!-- Includes -->
     <xacro:include filename="wheel.urdf.xacro"/>
@@ -52,7 +61,7 @@
         wheel_origin_xyz="0 0 0"
         wheel_origin_rpy="-${wheel_roll} ${wheel_pitch} ${wheel_yaw}"/>
-    <!-- Fixed joint to world -->
-    <joint name="world_to_link_body" type="fixed">
-        <parent link="world"/>
+    <!-- Fixed joint to link_base -->
+    <joint name="link_base_to_link_body" type="fixed">
+        <parent link="link_base"/>
         <child link="link_body"/>
         <origin xyz="0 0 0" rpy="0 0 0"/>

File: src/robot_description/urdf/wheel.urdf.xacro (robot description, xacro)
@@ -12,5 +12,11 @@
         </joint>
         <!-- Steering Link -->
-        <link name="link_steering_${wheel_name}" />
+        <link name="link_steering_${wheel_name}">
+            <inertial>
+                <origin xyz="0 0 0" rpy="0 0 0"/>
+                <mass value="1.0"/>
+                <inertia ixx="0.01" iyy="0.01" izz="0.01" ixy="0.0" ixz="0.0" iyz="0.0"/>
+            </inertial>
+        </link>
         <!-- Rotational Joint -->
         <joint name="joint_rotation_${wheel_name}" type="continuous">
@@ -27,5 +33,5 @@
                     <mesh filename="package://robot_description/meshes/tire.stl" scale="1.0 1.0 1.0"/>
                 </geometry>
-                <material name="color_body_front"/>
+                <material name="Black"/>
             </visual>
             <!-- Rims Mesh -->
@@ -34,5 +40,5 @@
                     <mesh filename="package://robot_description/meshes/rims.stl" scale="1.0 1.0 1.0"/>
                 </geometry>
-                <material name="color_body_front"/>
+                <material name="Black"/>
             </visual>
              <!-- Tire Mesh -->

Commit message: Update mass values in URDF files for body and wheel components

File: src/robot_description/urdf/body.urdf.xacro (robot description, xacro)
@@ -50,5 +50,5 @@
         <inertial>
             <origin xyz="0 0 0" rpy="0 0 0" />
-            <mass value="1.0" />
+            <mass value="50.0" />
             <inertia ixx="0.126164" ixy="0.0" ixz="0.0" iyy="0.416519" iyz="0.0" izz="0.481014" />
         </inertial>

File: src/robot_description/urdf/wheel.urdf.xacro (robot description, xacro)
@@ -57,5 +57,5 @@
             <inertial>
                 <origin xyz="0 0 0" rpy="0 0 0"/>
-                <mass value="2.0"/>
+                <mass value="10.0"/>
                 <inertia ixx="0.1" ixy="0.0" ixz="0.0" iyy="0.1" iyz="0.0" izz="0.1"/>
             </inertial>

Commit message: Refactor installation scripts for ROS2 compatibility, update mass and inertia values in URDF files, and enhance joystick speed control logic with exponential acceleration and deceleration.

File: src/robot_description/urdf/body.urdf.xacro (robot description, xacro)
@@ -1,4 +1,9 @@
 <?xml version="1.0"?>
 <robot xmlns:xacro="http://www.ros.org/wiki/xacro">
+    <!--
+    comprimento 597.271 mm
+    altura 138.91590 mm
+    largura 250.382 mm
+     -->
     <!-- Main body -->
     <link name="link_body">
@@ -50,6 +55,8 @@
         <inertial>
             <origin xyz="0 0 0" rpy="0 0 0" />
-            <mass value="50.0" />
+            <mass value="32.0" />
+            <!-- <inertia ixx="1.186" ixy="0.0" ixz="0.0" iyy="1.02" iyz="0.0" izz="5.18" /> -->
             <inertia ixx="0.126164" ixy="0.0" ixz="0.0" iyy="0.416519" iyz="0.0" izz="0.481014" />
+            <!-- <inertia ixx="8.125" ixy="0.0" ixz="0.0" iyy="30.625" iyz="0.0" izz="45.0" /> -->
         </inertial>
     </link>

File: src/robot_description/urdf/gazebo_control.xacro (robot description, xacro)
@@ -12,4 +12,20 @@
     </gazebo>
     <!-- Gazebo Wheels Ref -->
+    <!-- <gazebo reference="link_wheel_front_left">
+        <mu1 value="1.0"/>
+        <mu2 value="1.0"/>
+    </gazebo>
+    <gazebo reference="link_wheel_front_right">
+        <mu1 value="1.0"/>
+        <mu2 value="1.0"/>
+    </gazebo>
+    <gazebo reference="link_wheel_rear_left">
+        <mu1 value="1.0"/>
+        <mu2 value="1.0"/>
+    </gazebo>
+    <gazebo reference="link_wheel_rear_right">
+        <mu1 value="1.0"/>
+        <mu2 value="1.0"/>
+    </gazebo> -->
     <gazebo reference="link_wheel_front_left">
         <mu1 value="0.001"/>

File: src/robot_description/urdf/robot_core.xacro (robot description, xacro)
@@ -14,6 +14,12 @@
         <color rgba="1 1 1 1" />
     </material>
-    <!-- Root link_base -->fl_wheel_joint
-    <link name="link_base" />
+    <!-- Root link_base -->
+    <link name="link_base">
+        <inertial>
+            <origin xyz="0 0 0" rpy="0 0 0" />
+            <mass value="0.0" />
+            <inertia ixx="0.0" ixy="0.0" ixz="0.0" iyy="0.0" iyz="0.0" izz="0.0" />
+        </inertial>
+    </link>
     <!-- Includes -->
     <xacro:include filename="wheel.urdf.xacro"/>

File: src/robot_description/urdf/ros2_control.xacro (robot description, xacro)
@@ -23,6 +23,6 @@
       <joint name="joint_rotation_front_left">
         <command_interface name="velocity">
-          <param name="min">-10</param>
-          <param name="max">10</param>
+          <param name="min">-100</param>
+          <param name="max">100</param>
         </command_interface>
         <state_interface name="velocity"/>
@@ -30,6 +30,6 @@
       <joint name="joint_rotation_front_right">
         <command_interface name="velocity">
-          <param name="min">-10</param>
-          <param name="max">10</param>
+          <param name="min">-100</param>
+          <param name="max">100</param>
         </command_interface>
         <state_interface name="velocity"/>
@@ -37,6 +37,6 @@
       <joint name="joint_rotation_rear_left">
         <command_interface name="velocity">
-          <param name="min">-10</param>
-          <param name="max">10</param>
+          <param name="min">-100</param>
+          <param name="max">100</param>
         </command_interface>
         <state_interface name="velocity"/>
@@ -44,6 +44,6 @@
       <joint name="joint_rotation_rear_right">
         <command_interface name="velocity">
-          <param name="min">-10</param>
-          <param name="max">10</param>
+          <param name="min">-100</param>
+          <param name="max">100</param>
         </command_interface>
         <state_interface name="velocity"/>

File: src/robot_description/urdf/wheel.urdf.xacro (robot description, xacro)
@@ -57,6 +57,6 @@
             <inertial>
                 <origin xyz="0 0 0" rpy="0 0 0"/>
-                <mass value="10.0"/>
-                <inertia ixx="0.1" ixy="0.0" ixz="0.0" iyy="0.1" iyz="0.0" izz="0.1"/>
+                <mass value="5.0" />
+                <inertia ixx="0.1125" ixy="0.0" ixz="0.0" iyy="0.225" iyz="0.0" izz="0.1125" />
             </inertial>
         </link>

Commit message: Update URDF files: modify inertial properties for body and wheels, enhance wheel friction parameters, and adjust gazebo references

File: src/robot_description/urdf/body.urdf.xacro (robot description, xacro)
@@ -54,9 +54,8 @@
         <!-- Inertial -->
         <inertial>
-            <origin xyz="0 0 0" rpy="0 0 0" />
-            <mass value="32.0" />
-            <!-- <inertia ixx="1.186" ixy="0.0" ixz="0.0" iyy="1.02" iyz="0.0" izz="5.18" /> -->
-            <inertia ixx="0.126164" ixy="0.0" ixz="0.0" iyy="0.416519" iyz="0.0" izz="0.481014" />
-            <!-- <inertia ixx="8.125" ixy="0.0" ixz="0.0" iyy="30.625" iyz="0.0" izz="45.0" /> -->
+            <origin xyz="0 0 -0.1" rpy="0 0 0" />
+            <mass value="500.0" />
+            <inertia ixx="0.1" ixy="0.0" ixz="0.0" iyy="0.1" iyz="0.0" izz="0.1" />
+            <!-- <inertia ixx="0.126164" ixy="0.0" ixz="0.0" iyy="0.416519" iyz="0.0" izz="0.481014" /> -->
         </inertial>
     </link>

File: src/robot_description/urdf/gazebo_control.xacro (robot description, xacro)
@@ -9,23 +9,34 @@
     </gazebo>
     <!-- Gazebo Body Ref -->
-    <gazebo reference="link_body">
+    <!-- Gazebo Wheels Ref -->
+    <!-- <gazebo reference="link_body">
+        <kp>500.0</kp>
+        <kd>50.0</kd>
     </gazebo>
-    <!-- Gazebo Wheels Ref -->
-    <!-- <gazebo reference="link_wheel_front_left">
-        <mu1 value="1.0"/>
-        <mu2 value="1.0"/>
+    <gazebo reference="link_wheel_front_left">
+        <mu1 value="2.5"/>
+        <mu2 value="2.5"/>
+        <spring_k>10000</spring_k>
+        <damping>500</damping>
     </gazebo>
     <gazebo reference="link_wheel_front_right">
-        <mu1 value="1.0"/>
-        <mu2 value="1.0"/>
+        <mu1 value="2.5"/>
+        <mu2 value="2.5"/>
+        <spring_k>10000</spring_k>
+        <damping>500</damping>
     </gazebo>
     <gazebo reference="link_wheel_rear_left">
-        <mu1 value="1.0"/>
-        <mu2 value="1.0"/>
+        <mu1 value="2.5"/>
+        <mu2 value="2.5"/>
+        <spring_k>10000</spring_k>
+        <damping>500</damping>
     </gazebo>
     <gazebo reference="link_wheel_rear_right">
-        <mu1 value="1.0"/>
-        <mu2 value="1.0"/>
-    </gazebo> -->
+        <mu1 value="2.5"/>
+        <mu2 value="2.5"/>
+        <spring_k>10000</spring_k>
+        <damping>500</damping>
+    </gazebo>
+ -->
     <gazebo reference="link_wheel_front_left">
         <mu1 value="0.001"/>

File: src/robot_description/urdf/wheel.urdf.xacro (robot description, xacro)
@@ -57,6 +57,6 @@
             <inertial>
                 <origin xyz="0 0 0" rpy="0 0 0"/>
-                <mass value="5.0" />
-                <inertia ixx="0.1125" ixy="0.0" ixz="0.0" iyy="0.225" iyz="0.0" izz="0.1125" />
+                <mass value="25.0" />
+                <inertia ixx="0.00669" ixy="0.0" ixz="0.0" iyy="0.01154" iyz="0.0" izz="0.01154" />
             </inertial>
         </link>

Commit message: Revert "Update URDF files: modify inertial properties for body and wheels, enhance wheel friction parameters, and adjust gazebo references"
This reverts commit 2f7c3f8c955c7101f9b4b7112a1868460bc5991b.

File: src/robot_description/urdf/body.urdf.xacro (robot description, xacro)
@@ -54,8 +54,9 @@
         <!-- Inertial -->
         <inertial>
-            <origin xyz="0 0 -0.1" rpy="0 0 0" />
-            <mass value="500.0" />
-            <inertia ixx="0.1" ixy="0.0" ixz="0.0" iyy="0.1" iyz="0.0" izz="0.1" />
-            <!-- <inertia ixx="0.126164" ixy="0.0" ixz="0.0" iyy="0.416519" iyz="0.0" izz="0.481014" /> -->
+            <origin xyz="0 0 0" rpy="0 0 0" />
+            <mass value="32.0" />
+            <!-- <inertia ixx="1.186" ixy="0.0" ixz="0.0" iyy="1.02" iyz="0.0" izz="5.18" /> -->
+            <inertia ixx="0.126164" ixy="0.0" ixz="0.0" iyy="0.416519" iyz="0.0" izz="0.481014" />
+            <!-- <inertia ixx="8.125" ixy="0.0" ixz="0.0" iyy="30.625" iyz="0.0" izz="45.0" /> -->
         </inertial>
     </link>

File: src/robot_description/urdf/gazebo_control.xacro (robot description, xacro)
@@ -9,34 +9,23 @@
     </gazebo>
     <!-- Gazebo Body Ref -->
+    <gazebo reference="link_body">
+    </gazebo>
     <!-- Gazebo Wheels Ref -->
-    <!-- <gazebo reference="link_body">
-        <kp>500.0</kp>
-        <kd>50.0</kd>
-    </gazebo>
-    <gazebo reference="link_wheel_front_left">
-        <mu1 value="2.5"/>
-        <mu2 value="2.5"/>
-        <spring_k>10000</spring_k>
-        <damping>500</damping>
+    <!-- <gazebo reference="link_wheel_front_left">
+        <mu1 value="1.0"/>
+        <mu2 value="1.0"/>
     </gazebo>
     <gazebo reference="link_wheel_front_right">
-        <mu1 value="2.5"/>
-        <mu2 value="2.5"/>
-        <spring_k>10000</spring_k>
-        <damping>500</damping>
+        <mu1 value="1.0"/>
+        <mu2 value="1.0"/>
     </gazebo>
     <gazebo reference="link_wheel_rear_left">
-        <mu1 value="2.5"/>
-        <mu2 value="2.5"/>
-        <spring_k>10000</spring_k>
-        <damping>500</damping>
+        <mu1 value="1.0"/>
+        <mu2 value="1.0"/>
     </gazebo>
     <gazebo reference="link_wheel_rear_right">
-        <mu1 value="2.5"/>
-        <mu2 value="2.5"/>
-        <spring_k>10000</spring_k>
-        <damping>500</damping>
-    </gazebo>
- -->
+        <mu1 value="1.0"/>
+        <mu2 value="1.0"/>
+    </gazebo> -->
     <gazebo reference="link_wheel_front_left">
         <mu1 value="0.001"/>

File: src/robot_description/urdf/wheel.urdf.xacro (robot description, xacro)
@@ -57,6 +57,6 @@
             <inertial>
                 <origin xyz="0 0 0" rpy="0 0 0"/>
-                <mass value="25.0" />
-                <inertia ixx="0.00669" ixy="0.0" ixz="0.0" iyy="0.01154" iyz="0.0" izz="0.01154" />
+                <mass value="5.0" />
+                <inertia ixx="0.1125" ixy="0.0" ixz="0.0" iyy="0.225" iyz="0.0" izz="0.1125" />
             </inertial>
         </link>

Commit message: Revert "Refactor installation scripts for ROS2 compatibility, update mass and inertia values in URDF files, and enhance joystick speed control logic with exponential acceleration and deceleration."
This reverts commit 602ec28b740f2eb6fdfbe0648270b69624631220.

File: src/robot_description/urdf/body.urdf.xacro (robot description, xacro)
@@ -1,9 +1,4 @@
 <?xml version="1.0"?>
 <robot xmlns:xacro="http://www.ros.org/wiki/xacro">
-    <!--
-    comprimento 597.271 mm
-    altura 138.91590 mm
-    largura 250.382 mm
-     -->
     <!-- Main body -->
     <link name="link_body">
@@ -55,8 +50,6 @@
         <inertial>
             <origin xyz="0 0 0" rpy="0 0 0" />
-            <mass value="32.0" />
-            <!-- <inertia ixx="1.186" ixy="0.0" ixz="0.0" iyy="1.02" iyz="0.0" izz="5.18" /> -->
+            <mass value="50.0" />
             <inertia ixx="0.126164" ixy="0.0" ixz="0.0" iyy="0.416519" iyz="0.0" izz="0.481014" />
-            <!-- <inertia ixx="8.125" ixy="0.0" ixz="0.0" iyy="30.625" iyz="0.0" izz="45.0" /> -->
         </inertial>
     </link>

File: src/robot_description/urdf/gazebo_control.xacro (robot description, xacro)
@@ -12,20 +12,4 @@
     </gazebo>
     <!-- Gazebo Wheels Ref -->
-    <!-- <gazebo reference="link_wheel_front_left">
-        <mu1 value="1.0"/>
-        <mu2 value="1.0"/>
-    </gazebo>
-    <gazebo reference="link_wheel_front_right">
-        <mu1 value="1.0"/>
-        <mu2 value="1.0"/>
-    </gazebo>
-    <gazebo reference="link_wheel_rear_left">
-        <mu1 value="1.0"/>
-        <mu2 value="1.0"/>
-    </gazebo>
-    <gazebo reference="link_wheel_rear_right">
-        <mu1 value="1.0"/>
-        <mu2 value="1.0"/>
-    </gazebo> -->
     <gazebo reference="link_wheel_front_left">
         <mu1 value="0.001"/>

File: src/robot_description/urdf/robot_core.xacro (robot description, xacro)
@@ -14,12 +14,6 @@
         <color rgba="1 1 1 1" />
     </material>
-    <!-- Root link_base -->
-    <link name="link_base">
-        <inertial>
-            <origin xyz="0 0 0" rpy="0 0 0" />
-            <mass value="0.0" />
-            <inertia ixx="0.0" ixy="0.0" ixz="0.0" iyy="0.0" iyz="0.0" izz="0.0" />
-        </inertial>
-    </link>
+    <!-- Root link_base -->fl_wheel_joint
+    <link name="link_base" />
     <!-- Includes -->
     <xacro:include filename="wheel.urdf.xacro"/>

File: src/robot_description/urdf/ros2_control.xacro (robot description, xacro)
@@ -23,6 +23,6 @@
       <joint name="joint_rotation_front_left">
         <command_interface name="velocity">
-          <param name="min">-100</param>
-          <param name="max">100</param>
+          <param name="min">-10</param>
+          <param name="max">10</param>
         </command_interface>
         <state_interface name="velocity"/>
@@ -30,6 +30,6 @@
       <joint name="joint_rotation_front_right">
         <command_interface name="velocity">
-          <param name="min">-100</param>
-          <param name="max">100</param>
+          <param name="min">-10</param>
+          <param name="max">10</param>
         </command_interface>
         <state_interface name="velocity"/>
@@ -37,6 +37,6 @@
       <joint name="joint_rotation_rear_left">
         <command_interface name="velocity">
-          <param name="min">-100</param>
-          <param name="max">100</param>
+          <param name="min">-10</param>
+          <param name="max">10</param>
         </command_interface>
         <state_interface name="velocity"/>
@@ -44,6 +44,6 @@
       <joint name="joint_rotation_rear_right">
         <command_interface name="velocity">
-          <param name="min">-100</param>
-          <param name="max">100</param>
+          <param name="min">-10</param>
+          <param name="max">10</param>
         </command_interface>
         <state_interface name="velocity"/>

File: src/robot_description/urdf/wheel.urdf.xacro (robot description, xacro)
@@ -57,6 +57,6 @@
             <inertial>
                 <origin xyz="0 0 0" rpy="0 0 0"/>
-                <mass value="5.0" />
-                <inertia ixx="0.1125" ixy="0.0" ixz="0.0" iyy="0.225" iyz="0.0" izz="0.1125" />
+                <mass value="10.0"/>
+                <inertia ixx="0.1" ixy="0.0" ixz="0.0" iyy="0.1" iyz="0.0" izz="0.1"/>
             </inertial>
         </link>

Commit message: Enhance teleop launch file with terminal instructions, update URDF inertial properties, improve wheel friction parameters, and refine installation scripts for ROS2 compatibility.

File: src/robot_description/urdf/body.urdf.xacro (robot description, xacro)
@@ -1,4 +1,9 @@
 <?xml version="1.0"?>
 <robot xmlns:xacro="http://www.ros.org/wiki/xacro">
+     <!--
+    comprimento 597.271 mm
+    altura 138.91590 mm
+    largura 250.382 mm
+     -->
     <!-- Main body -->
     <link name="link_body">
@@ -49,7 +54,7 @@
         <!-- Inertial -->
         <inertial>
-            <origin xyz="0 0 0" rpy="0 0 0" />
-            <mass value="50.0" />
-            <inertia ixx="0.126164" ixy="0.0" ixz="0.0" iyy="0.416519" iyz="0.0" izz="0.481014" />
+            <origin xyz="0 0 -0.11" rpy="0 0 0" />
+            <mass value="28.0" />
+            <inertia ixx="0.1913" ixy="0.0" ixz="0.0" iyy="0.9787" iyz="0.0" izz="0.8774" />
         </inertial>
     </link>

File: src/robot_description/urdf/gazebo_control.xacro (robot description, xacro)
@@ -13,18 +13,18 @@
     <!-- Gazebo Wheels Ref -->
     <gazebo reference="link_wheel_front_left">
-        <mu1 value="0.001"/>
-        <mu2 value="0.001"/>
+        <mu1 value="0.005"/>
+        <mu2 value="0.005"/>
     </gazebo>
     <gazebo reference="link_wheel_front_right">
-        <mu1 value="0.001"/>
-        <mu2 value="0.001"/>
+        <mu1 value="0.005"/>
+        <mu2 value="0.005"/>
     </gazebo>
     <gazebo reference="link_wheel_rear_left">
-        <mu1 value="0.001"/>
-        <mu2 value="0.001"/>
+        <mu1 value="0.005"/>
+        <mu2 value="0.005"/>
     </gazebo>
     <gazebo reference="link_wheel_rear_right">
-        <mu1 value="0.001"/>
-        <mu2 value="0.001"/>
+        <mu1 value="0.005"/>
+        <mu2 value="0.005"/>
     </gazebo>
 </robot>
