Commit message: Refactor motor control parameters, update URDF limits, and add new Arduino script for ROS2 communication

File: src/robot_description/urdf/ros2_control.xacro (robot description, xacro)
@@ -16,5 +16,5 @@
             <param name="rear_wheel_right_pos">joint_steering_rear_right</param>
             <param name="rear_wheel_left_pos">joint_steering_rear_left</param>
-            <param name="device">/dev/ttyACM0</param>
+            <param name="device">/dev/ttyUSB0</param>
             <param name="baud_rate">115200</param>
             <param name="timeout_ms">1000</param>

File: src/robot_description/urdf/wheel.urdf.xacro (robot description, xacro)
@@ -9,5 +9,5 @@
             <axis xyz="${steering_axis_xyz}"/>
             <origin xyz="${steering_origin_xyz}" rpy="${steering_origin_rpy}"/>
-            <limit effort="10.0" velocity="1.0" lower="-0.45" upper="0.45"/>
+            <limit effort="10.0" velocity="1.0" lower="-0.523598333" upper="0.523598333"/> <!-- -30 to 30 degrees -->
         </joint>
         <!-- Steering Link -->
